Commit message: switch from camera to Asus Xtion in URDF file

File: simulation_tobot/beebot_description/urdf/beebot.xacro (robot description, xacro)
@@ -136,33 +136,9 @@
   <xacro:fb_wheel prefix="front" reflect="1"/>
   <xacro:fb_wheel prefix="back" reflect="-1"/>
-  <!--CAMERA-->
-  <link name="camera_link">
-    <visual>
-      <geometry>
-        <box size="0.035 0.178 0.024"/>
-      </geometry>
-      <origin rpy="0 0 0" xyz="0 0 0"/>
-      <material name="black"/>
-    </visual>
-    <collision>
-      <origin xyz="0 0 0" rpy="0 0 0" />
-      <geometry>
-          <box size="0.035 0.185 0.025"/>
-      </geometry>
-    </collision>
-    <inertial>
-        <mass value="0.200" />
-        <origin xyz="0 0 0" />
-        <inertia ixx="5.8083e-4" ixy="0" ixz="0"
-                 iyy="3.0833e-5" iyz="0"
-                 izz="5.9083e-4" />
-    </inertial>
-  </link>
-  <joint name="camera" type="fixed">
-    <parent link="base_link"/>
-    <child link="camera_link"/>
-    <!--<origin xyz="${width} 0 ${GROUND_CLEARANCE-bodylen+posz_camera} " rpy="0 0 0"/>-->
+  <!--Asus Xtion sensor -->
+  <xacro:include filename="$(find hector_sensors_description)/urdf/asus_camera.urdf.xacro" />
+  <xacro:asus_camera name="camera" parent="base_link">
     <origin xyz="${width + 0.07} 0 0.05 " rpy="0 0 0"/>
-  </joint>
+  </xacro:asus_camera>
   <!--LASER-->
   <link name="hokuyo_link">

Commit message: Fixed goal publisher's bug and adjust some parameters for simulation purpose

File: simulation_tobot/beebot_description/urdf/beebot.xacro (robot description, xacro)
@@ -6,15 +6,15 @@
   <xacro:property name="GROUND_CLEARANCE" value="0.0335" />
   <xacro:property name="width" value="0.40" />
-  <xacro:property name="xpsvwhloffset" value="0.3374" />
-  <xacro:property name="yactwhloffset" value="0.4238" />
+  <xacro:property name="xpsvwhloffset" value="0.230" />
+  <xacro:property name="yactwhloffset" value="0.25805" />
   <xacro:property name="bodylen" value="0.355" />
   <xacro:property name="wheel_w" value="0.039" />
-  <xacro:property name="wheel_rad" value="0.1194" />
-  <xacro:property name="plat_rad" value="0.3" />
+  <xacro:property name="wheel_rad" value="0.075" />
+  <xacro:property name="plat_rad" value="0.42" />
   <xacro:property name="plat_len" value="0.005" />
   <xacro:property name="HIGH_PLATFORM" value="0.15" />
-  <xacro:property name="posz_laser" value="0.285" />
-  <xacro:property name="posz_camera" value="0.5" />
-  <xacro:property name="fwheel_rad" value="0.08276" />
+  <xacro:property name="posz_laser" value="0.118" />
+  <xacro:property name="posz_camera" value="0.2485" />
+  <xacro:property name="fwheel_rad" value="0.0376094" />
   <xacro:property name="pi" value="3.1415" />
   <!--Mass values for each link in kg-->
@@ -139,5 +139,6 @@
   <xacro:include filename="$(find hector_sensors_description)/urdf/asus_camera.urdf.xacro" />
   <xacro:asus_camera name="camera" parent="base_link">
-    <origin xyz="${width + 0.07} 0 0.05 " rpy="0 0 0"/>
+    <!--<origin xyz="${width + 0.07} 0 0.05 " rpy="0 0 0"/>-->
+    <origin xyz="${width} 0 ${posz_camera}" rpy="0 0 0" />
   </xacro:asus_camera>
   <!--LASER-->
@@ -168,5 +169,6 @@
     <parent link="base_link"/>
     <child link="hokuyo_link"/>
-    <origin xyz="${width + 0.07} 0 ${GROUND_CLEARANCE-bodylen+posz_laser} " rpy="0 0 0"/>
+    <!--<origin xyz="${width + 0.07} 0 ${GROUND_CLEARANCE-bodylen+posz_laser} " rpy="0 0 0"/>-->
+    <origin xyz="${width} 0 ${posz_laser}" rpy="0 0 0" />
   </joint>
 </robot>
